File: hardware/motor-control-board/circuit/V2_PH/motor-controller-pcb/motor-controller-pcb.kicad_pcb (KiCad board)
At the start: 4 copper layers, 50 x 70 mm, 61 parts, among them J1 USB-C Power, J2 Motor Conn, J3 NEMA17, J4 OLED Screen, J5 Motor Conn, J6 NEMA17, J7 GPIO, J8 SG90, Q1 DP2101W, Q2 WST2011, SW1 SW_Push, SW3 MST22D18G2 125, U1 DRV8428RTER, U2 FP6291LR-G1, U2 RP2040 XIAO, U3 DRV8428RTER

Commit message: PCB ready for manufacture
Parts:
- removed the H1 at (107.9, 63.4)
- removed the H2 at (107.9, 125.8)
- removed the U2 at (121.9, 56.3)
- added H5: M3, MountingHole:MountingHole_3.2mm_M3, F.Cu at (127.1, 100.8)
- added H6: M3, MountingHole:MountingHole_3.2mm_M3, F.Cu at (127.0, 123.0)
- added JP1: Jumper_3_Bridged12, blot-footprints:JUMPER-3Psml_Bridged_RoundedPad2x1mm, F.Cu at (117.3, 100.1)
- added JP2: Jumper_3_Bridged12, blot-footprints:JUMPER-3Psml_Bridged_RoundedPad2x1mm, F.Cu at (117.0, 121.6)
- added U4: RP2040 XIAO, blot-footprints:QTPYXIAORP2040, F.Cu at (121.9, 56.3)
- F1: value 600mA -> 800mA
- J2: renamed from J4; footprint Connector_PinHeader_2.54mm:PinHeader_1x04_P2.54mm_Vertical -> Connector_PinSocket_2.54mm:PinSocket_1x04_P2.54mm_Vertical
- J4: renamed from J3; footprint Connector_PinHeader_2.54mm:PinHeader_1x04_P2.54mm_Vertical -> Connector_PinSocket_2.54mm:PinSocket_1x04_P2.54mm_Vertical
- J6: renamed from J8; footprint Connector_PinHeader_2.54mm:PinHeader_1x03_P2.54mm_Vertical -> Connector_PinSocket_2.54mm:PinSocket_1x03_P2.54mm_Vertical
- J8: renamed from J6; footprint Connector_PinHeader_2.54mm:PinHeader_1x04_P2.54mm_Vertical -> Connector_PinSocket_2.54mm:PinSocket_1x04_P2.54mm_Vertical
- R13: renamed from R7; value 100K -> 60K
- SW2: renamed from SW1; value SW_Push -> User
- moved D2 29.1 mm to (106.3, 103.6), turned to 0 degrees
- moved D3 28.7 mm to (106.3, 107.1), turned to 0 degrees
- moved R9 25.0 mm to (109.3, 103.6), turned to 180 degrees
- moved R10 24.5 mm to (109.2, 107.1), turned to 180 degrees
- moved C6 11.2 mm to (141.7, 83.6), turned to 0 degrees
- moved C9 9.32 mm to (141.7, 85.1), turned to 180 degrees
- moved C11 8.40 mm to (142.2, 95.3), turned to 0 degrees
- moved R15 8.29 mm to (144.2, 91.2), turned to -90 degrees
- moved J2 7.62 mm to (150.4, 115.7), turned to 180 degrees
- moved R5 7.54 mm to (145.8, 115.7)
- moved R13 7.34 mm to (142.8, 88.2), turned to 90 degrees
- moved C12 6.91 mm to (142.2, 93.7), turned to 180 degrees
- moved R14 6.18 mm to (142.7, 91.2), turned to 90 degrees
- moved U2 4.60 mm to (140.3, 88.2), turned to -90 degrees
- moved L1 4.50 mm to (136.8, 88.0), turned to -90 degrees
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- renumbered C5 to C3, C3 to C4, C4 to C5, C7 to C6, C6 to C7, C9 to C8, C8 to C9, D4 to D1, D1 to D4, J2 to J3, Q2 to Q1, Q1 to Q2, R11 to R10, R6 to R11, R5 to R12, R8 to R14, R9 to R15, R12 to R16, R3 to R2, R4 to R3, R15 to R4, R16 to R5, R2 to R6, R14 to R7, R13 to R8, R10 to R9, SW3 to SW1
Connections:
- RV1 pad 2: Net-(U1-VREF) -> Net-(JP1-B)
- RV2 pad 2: Net-(U3-VREF) -> Net-(JP2-B)
- U1 pad 7: Net-(U1-VREF) -> Net-(JP1-C)
- U3 pad 7: Net-(U3-VREF) -> Net-(JP2-C)
Routing:
- net GND: track 0.00 -> 109.6 mm, vias 0 -> 91
- net VMEM: track 0.00 -> 84.4 mm, vias 0 -> 9
- net +5VA: track 13.4 -> 84.0 mm, vias 1 -> 7
- net /DAC: track 12.8 -> 82.4 mm, vias 0 -> 2
- net (no net): track 67.1 -> 0.05 mm, vias 1 -> 0
- net /SDA: track 10.2 -> 74.5 mm
- net /ENABLE: track 0.00 -> 58.7 mm
- net /SCL: track 10.2 -> 65.8 mm
- net /A2: track 10.2 -> 65.3 mm
- net /A8: track 0.00 -> 47.9 mm, vias 0 -> 1
- net /A7: track 0.00 -> 42.9 mm, vias 0 -> 1
- net /A6: track 0.00 -> 40.1 mm
- net /A10: track 0.00 -> 30.7 mm, vias 0 -> 1
- net /A9: track 0.00 -> 26.2 mm, vias 0 -> 1
- net VBUS: track 0.00 -> 22.2 mm, vias 0 -> 2
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- added copper zone on In2.Cu, net +3V3
- added copper zone on B.Cu, net GND
- added copper zone on F.Cu, net GND
- added copper zone on In1.Cu, net GND
- removed copper zone on B.Cu, net (none)
- removed copper zone on F.Cu, net (none)
Other:
- board text added: "3"
- board text added: "3V3"
- board text added: "5"
- board text added: "5V"
- board text added: "A2"
- board text added: "A3"
- board text added: "BLOT"
- board text added: "Board Dimensions: 50.00mm x 70.00mm FR4 1.6mm, 4-layer"
- board text added: "C"
- board text added: "D"
- board text added: "DAC"
- board text added: "Data"
- board text added: "G"
- board text added: "GND"
- board text added: "HACK CLUB"
- board text added: "M1"
- board text added: "M2"
- board text added: "M3"
- board text added: "OLED Display 128x64"
- board text added: "SCL"
- board text added: "SDA"
- board text added: "Servo"
- board text added: "USB C Data + Power"
- board text added: "USB C Power Only"
- board text added: "VM+"
- board text added: "v2.1b1"
- board text removed: "Board Dimensions: 50.00mm x 70.00mm FR4 1.6mm, 2-layer"
