File: hardware/motor-control-board/circuit/V2_PH/motor-controller-pcb/motor-controller-pcb.kicad_pcb (KiCad board)
At the start: 4 copper layers, 50 x 70 mm, 63 parts, among them J1 USB-C Power, J2 OLED Screen, J3 Motor Conn, J4 NEMA17, J5 Motor Conn, J6 SG90, J7 GPIO, J8 NEMA17, Q1 WST2011, Q2 DP2101W, SW1 MST22D18G2 125, SW2 User, U1 DRV8428RTER, U2 FP6291LR-G1, U3 DRV8428RTER, U4 RP2040 XIAO

Commit message: adding in new PWM/DAC design
Parts:
- added C1: 10uF, Capacitor_SMD:C_0603_1608Metric, F.Cu at (136.9, 105.3)
- added C2: 100nF, Capacitor_SMD:C_0603_1608Metric, F.Cu at (134.3, 111.4)
- added FB1: 150, Inductor_SMD:L_1206_3216Metric, F.Cu at (130.9, 109.5)
- added JP1: Jumper_2_Open, blot-footprints:JUMPER-2Psml_UnBridged_RoundedPad2x1mm, F.Cu at (136.6, 104.1)
- added JP2: Jumper_2_Open, blot-footprints:JUMPER-2Psml_UnBridged_RoundedPad2x1mm, F.Cu at (134.7, 114.0)
- added L1: 2.2uH, Inductor_SMD:L_0603_1608Metric, F.Cu at (133.8, 103.8)
- added R1: 16R, Resistor_SMD:R_0603_1608Metric, F.Cu at (133.8, 105.4)
- added TP1: TestPoint, TestPoint:TestPoint_THTPad_1.0x1.0mm_Drill0.5mm, F.Cu at (113.3, 101.5)
- added TP2: TestPoint, TestPoint:TestPoint_THTPad_1.0x1.0mm_Drill0.5mm, F.Cu at (105.2, 67.2)
- added TP4: TestPoint, TestPoint:TestPoint_THTPad_1.0x1.0mm_Drill0.5mm, F.Cu at (112.8, 123.3)
- added U1: DAC5571IDBVR, easyeda2kicad:SOT-23-6_L2.9-W1.6-P0.95-LS2.8-BR, F.Cu at (130.9, 112.7)
- C10: renamed from C7; value 100nF -> 100nF/16V
- C11: renamed from C8; value 10nF/35V -> 10nF/16V
- C13: renamed from C11; value 22uF -> 22uF/16V
- C14: renamed from C12; value 100nF -> 100nF/16V
- C15: renamed from C13; value 10nF/35V -> 10nF/16V
- C3: value 22uF -> 22uF/16V
- C4: renamed from C1; value 10nF/35V -> 10nF/16V
- C6: renamed from C4; value 10nF/35V -> 10nF/16V
- C8: renamed from C6; value 22uF -> 22uF/16V
- C9: value 100nF -> 100nF/16V
- D3: value Green -> Emerald
- F1: value 800mA -> 1A
- Q2: value DP2101W -> HXY2101EI
- R12: renamed from R13; value 60K -> 60.4K
- R15: renamed from R14; value 168K -> 169K
- R2, R3, R4, R5, R8: footprint Resistor_SMD:R_0603_1608Metric_Pad0.98x0.95mm_HandSolder -> Resistor_SMD:R_0603_1608Metric
- renumbered C10 to C12, C14 to C16, C2 to C5, C5 to C7, J6 to J5, J7 to J6, J5 to J7, JP1 to JP3, JP2 to JP4, L1 to L2, R9 to R10, R10 to R11, R12 to R13, R11 to R14, R15 to R16, R16 to R17, R1 to R6, R6 to R9, TP1 to TP3, U1 to U2, U2 to U3, U3 to U5
Connections:
- JP3 pad 1: /DAC -> Vref1
- JP4 pad 1: /DAC -> Vref1
Routing:
- net Vref1: track 0.00 -> 64.6 mm, vias 0 -> 2
- net /SDA: track 74.5 -> 102.8 mm, vias 0 -> 1
- net /SCL: track 65.8 -> 90.6 mm, vias 0 -> 1
- net /DAC: track 82.4 -> 68.5 mm, vias 2 -> 1
- net GND: track 109.6 -> 117.1 mm, vias 91 -> 93
- net Net-(JP3-C): track 2.96 -> 10.1 mm
- net Net-(JP4-C): track 2.84 -> 8.74 mm, vias 0 -> 1
- net Net-(U1-VDD): track 0.00 -> 4.70 mm
- net Net-(JP1-A): track 0.00 -> 3.07 mm
- net +3V3: track 3.45 -> 6.03 mm, vias 4 -> 5
- net Net-(L1-Pad1): track 0.00 -> 2.25 mm
- net Net-(JP2-A): track 0.00 -> 1.97 mm
Other:
- board text added: "Vref"
