File: hardware/motor-control-board/circuit/V2_PH/motor-controller-pcb/motor-controller-pcb.kicad_sch (KiCad schematic)
At the start: 59 parts, among them J1 USB-C Power, J2 Motor Conn, J3 NEMA17, J4 OLED Screen, J5 Motor Conn, J6 NEMA17, J7 GPIO, J8 SG90, Q1 DP2101W, Q2 WST2011, SW1 User, SW3 MST22D18G2 125, U1 DRV8428RTER, U2 FP6291LR-G1, U3 DRV8428RTER, U4 RP2040 XIAO

Commit message: PCB ready for manufacture
Parts:
- added H5, H6: M3, MountingHole:MountingHole_3.2mm_M3, symbol Mechanical:MountingHole
- added JP1, JP2: Jumper_3_Bridged12, blot-footprints:JUMPER-3Psml_Bridged_RoundedPad2x1mm, symbol Jumper:Jumper_3_Bridged12
- F1: value 600mA -> 800mA
- J2: renamed from J4; footprint Connector_PinHeader_2.54mm:PinHeader_1x04_P2.54mm_Vertical -> Connector_PinSocket_2.54mm:PinSocket_1x04_P2.54mm_Vertical
- J4: renamed from J3; footprint Connector_PinHeader_2.54mm:PinHeader_1x04_P2.54mm_Vertical -> Connector_PinSocket_2.54mm:PinSocket_1x04_P2.54mm_Vertical
- J6: renamed from J8; footprint Connector_PinHeader_2.54mm:PinHeader_1x03_P2.54mm_Vertical -> Connector_PinSocket_2.54mm:PinSocket_1x03_P2.54mm_Vertical
- J8: renamed from J6; footprint Connector_PinHeader_2.54mm:PinHeader_1x04_P2.54mm_Vertical -> Connector_PinSocket_2.54mm:PinSocket_1x04_P2.54mm_Vertical
- RV1, RV2: now not fitted; now left out of the parts list
- U4: footprint Blot:QTPYXIAORP2040 -> blot-footprints:QTPYXIAORP2040
- renumbered C5 to C3, C3 to C4, C4 to C5, C7 to C6, C6 to C7, C9 to C8, C8 to C9, D4 to D1, D1 to D4, J2 to J3, Q2 to Q1, Q1 to Q2, R11 to R10, R6 to R11, R5 to R12, R7 to R13, R8 to R14, R9 to R15, R12 to R16, R3 to R2, R4 to R3, R15 to R4, R16 to R5, R2 to R6, R14 to R7, R13 to R8, R10 to R9, SW3 to SW1, SW1 to SW2
Connections:
- net DAC: now also JP1.1 (A), JP2.1 (A)
- net at U3.7 (VREF): now also JP2.2 (C); no longer RV2.2
- net at U1.7 (VREF): now also JP1.2 (C); no longer RV1.2
- new net: JP2.3 (B), RV2.2
- new net: JP1.3 (B), RV1.2
Other:
- note added: "PCB Tests: * check max motor current vs. 5V draw * is DC PSU OC resistor rating correct? What should it be? * after check above, check polyfuse rating"
- moved on the sheet: H1, H2, H3, H4
