File: hardware/motor-control-board/circuit/V2_PH/motor-controller-pcb/motor-controller-pcb.kicad_sch (KiCad schematic)
At the start: 63 parts, among them J1 USB-C Power, J2 OLED Screen, J3 Motor Conn, J4 NEMA17, J5 Motor Conn, J6 SG90, J7 GPIO, J8 NEMA17, Q1 WST2011, Q2 DP2101W, SW1 MST22D18G2 125, SW2 User, U1 DRV8428RTER, U2 FP6291LR-G1, U3 DRV8428RTER, U4 RP2040 XIAO

Commit message: updated components with LCSC part numbers
Parts:
- C1, C13, C4, C8: value 10nF/35V -> 10nF/16V; LCSC (none) -> C519406
- C10, C2: LCSC (none) -> C106851
- C11, C3, C6: value 22uF -> 22uF/16V; LCSC C30926 -> C6119868
- C12, C7, C9: value 100nF -> 100nF/16V
- D1, D4: LCSC (none) -> C2943878
- D2: LCSC (none) -> C965800
- D3: value Green -> Emerald; LCSC (none) -> C965804
- F1: value 800mA -> 1A; LCSC (none) -> C269104
- H1, H2, H3, H4, H5, H6, JP1, JP2, TP1, U4: LCSC (none) -> X
- J1: LCSC (none) -> C2765186
- J4, J8: LCSC (none) -> C2845390
- J6: LCSC (none) -> C2937625
- L1: LCSC (none) -> C5159366
- Q1: LCSC (none) -> C148368
- Q2: value DP2101W -> HXY2101EI; LCSC (none) -> C5148643; LCSC Part C2931644 -> C5148643
- R1, R11: LCSC (none) -> C22843
- R10: LCSC (none) -> C114612
- R13: value 60K -> 60.4K; LCSC (none) -> C23089
- R14: value 168K -> 169K; LCSC (none) -> C137791
- R15: LCSC (none) -> C22790
- R2, R3, R4, R5: footprint Resistor_SMD:R_0603_1608Metric_Pad0.98x0.95mm_HandSolder -> Resistor_SMD:R_0603_1608Metric; LCSC (none) -> C23186
- R7: LCSC (none) -> C14675
- R8: footprint Resistor_SMD:R_0603_1608Metric_Pad0.98x0.95mm_HandSolder -> Resistor_SMD:R_0603_1608Metric; LCSC (none) -> C14675
- R9: LCSC (none) -> C98220
- RV1, RV2: LCSC (none) -> C6331330
- SW1: LCSC (none) -> C2906280
- SW2: LCSC C318886 -> C843665
- U1, U3: LCSC (none) -> C2857955
- U2: LCSC (none) -> C18701

Commit message: adding in new PWM/DAC design
Parts:
- added C1: 10uF, Capacitor_SMD:C_0603_1608Metric, symbol Device:C_Small
- added C2: 100nF, Capacitor_SMD:C_0603_1608Metric, symbol Device:C_Small
- added FB1: 150, Inductor_SMD:L_1206_3216Metric, symbol Device:FerriteBead_Small
- added JP1, JP2: Jumper_2_Open, blot-footprints:JUMPER-2Psml_UnBridged_RoundedPad2x1mm, symbol Jumper:Jumper_2_Open
- added L1: 2.2uH, Inductor_SMD:L_0603_1608Metric, symbol Device:L_Small
- added R1: 16R, Resistor_SMD:R_0603_1608Metric, symbol Device:R_Small
- added TP1, TP2, TP4: TestPoint, TestPoint:TestPoint_THTPad_1.0x1.0mm_Drill0.5mm, symbol Connector:TestPoint
- added U1: DAC5571IDBVR, easyeda2kicad:SOT-23-6_L2.9-W1.6-P0.95-LS2.8-BR, symbol easyeda2kicad:DAC5571IDBVR
- renumbered C7 to C10, C8 to C11, C10 to C12, C11 to C13, C12 to C14, C13 to C15, C14 to C16, C1 to C4, C2 to C5, C4 to C6, C5 to C7, C6 to C8, J6 to J5, J7 to J6, J5 to J7, JP1 to JP3, JP2 to JP4, L1 to L2, R9 to R10, R10 to R11, R13 to R12, R12 to R13, R11 to R14, R14 to R15, R15 to R16, R16 to R17, R1 to R6, R6 to R9, TP1 to TP3, U1 to U2, U2 to U3, U3 to U5
Connections:
- net +3V3: now also FB1.1
- net DAC: now also R1.1; no longer JP3.1 (A), JP4.1 (A)
- net GND: now also C1.2, C2.2, TP2.1, U1.2 (GND), U1.6 (A0)
- net SCL: now also U1.5 (SCL)
- net SDA: now also U1.4 (SDA)
- net at JP4.2 (C), U5.7 (VREF): now also TP4.1
- net at JP3.2 (C), U2.7 (VREF): now also TP1.1
- new net: JP2.1 (A), U1.1 (VOUT)
- new net: C2.1, FB1.2, U1.3 (VDD)
- new net: L1.1, R1.2
- new net: C1.1, JP1.1 (A), L1.2
- new net Vref1: JP1.2 (B), JP2.2 (B), JP3.1 (A), JP4.1 (A)
Other:
- note added: "8-Bit DAC (0-5V)"
- note added: "Full tech using i2C DAC"
- note added: "Low tech using filtered low pass PWM"
- note added: "Note: DVDD is 5V i2C is 3.3V! Needs testing!"
- note added: "Vref"
- note added: "i2C Add: 0x4C or 0x4D"
- note added: "or 47R"
- moved on the sheet: C10, C11, C12, C13, C14, C15, C16, C3, C4, C5, C6, C7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
